File: Keep-KiCad/keeboard/keeboard.kicad_pcb (KiCad board)
At the start: 2 copper layers, 0 parts

Commit message: pcb edit & schematic
Parts:
- added D1: 1N4148, Diode_THT:D_DO-35_SOD27_P7.62mm_Horizontal, B.Cu at (153.5, 113.3)
- added D10: 1N4148, Diode_THT:D_DO-35_SOD27_P7.62mm_Horizontal, B.Cu at (344.0, 113.3)
- added D100: 1N4148, Diode_THT:D_DO-35_SOD27_P7.62mm_Horizontal, B.Cu at (405.9, 218.1)
- added D101: 1N4148, Diode_THT:D_DO-35_SOD27_P7.62mm_Horizontal, B.Cu at (425.0, 218.1)
- added D102: 1N4148, Diode_THT:D_DO-35_SOD27_P7.62mm_Horizontal, B.Cu at (444.0, 218.1)
- added D103: 1N4148, Diode_THT:D_DO-35_SOD27_P7.62mm_Horizontal, B.Cu at (477.4, 218.1)
- added D104: 1N4148, Diode_THT:D_DO-35_SOD27_P7.62mm_Horizontal, B.Cu at (506.0, 218.1)
- added D11: 1N4148, Diode_THT:D_DO-35_SOD27_P7.62mm_Horizontal, B.Cu at (363.1, 113.3)
- added D12: 1N4148, Diode_THT:D_DO-35_SOD27_P7.62mm_Horizontal, B.Cu at (382.1, 113.3)
- added D13: 1N4148, Diode_THT:D_DO-35_SOD27_P7.62mm_Horizontal, B.Cu at (405.9, 113.3)
- added D14: 1N4148, Diode_THT:D_DO-35_SOD27_P7.62mm_Horizontal, B.Cu at (425.0, 113.3)
- added D15: 1N4148, Diode_THT:D_DO-35_SOD27_P7.62mm_Horizontal, B.Cu at (444.0, 113.3)
- added D16: 1N4148, Diode_THT:D_DO-35_SOD27_P7.62mm_Horizontal, B.Cu at (115.4, 141.9)
- added D17: 1N4148, Diode_THT:D_DO-35_SOD27_P7.62mm_Horizontal, B.Cu at (134.5, 141.9)
- added D18: 1N4148, Diode_THT:D_DO-35_SOD27_P7.62mm_Horizontal, B.Cu at (153.5, 141.9)
- added D19: 1N4148, Diode_THT:D_DO-35_SOD27_P7.62mm_Horizontal, B.Cu at (172.6, 141.9)
- added D2: 1N4148, Diode_THT:D_DO-35_SOD27_P7.62mm_Horizontal, B.Cu at (172.6, 113.3)
- added D20: 1N4148, Diode_THT:D_DO-35_SOD27_P7.62mm_Horizontal, B.Cu at (191.6, 141.9)
- added D21: 1N4148, Diode_THT:D_DO-35_SOD27_P7.62mm_Horizontal, B.Cu at (210.7, 141.9)
- added D22: 1N4148, Diode_THT:D_DO-35_SOD27_P7.62mm_Horizontal, B.Cu at (229.7, 141.9)
- added D23: 1N4148, Diode_THT:D_DO-35_SOD27_P7.62mm_Horizontal, B.Cu at (248.8, 141.9)
- added D24: 1N4148, Diode_THT:D_DO-35_SOD27_P7.62mm_Horizontal, B.Cu at (267.8, 141.9)
- added D25: 1N4148, Diode_THT:D_DO-35_SOD27_P7.62mm_Horizontal, B.Cu at (286.9, 141.9)
- added D26: 1N4148, Diode_THT:D_DO-35_SOD27_P7.62mm_Horizontal, B.Cu at (305.9, 141.9)
- added D27: 1N4148, Diode_THT:D_DO-35_SOD27_P7.62mm_Horizontal, B.Cu at (325.0, 141.9)
- added D28: 1N4148, Diode_THT:D_DO-35_SOD27_P7.62mm_Horizontal, B.Cu at (344.0, 141.9)
- added D29: 1N4148, Diode_THT:D_DO-35_SOD27_P7.62mm_Horizontal, B.Cu at (372.6, 141.9)
- added D3: 1N4148, Diode_THT:D_DO-35_SOD27_P7.62mm_Horizontal, B.Cu at (191.6, 113.3)
- added D30: 1N4148, Diode_THT:D_DO-35_SOD27_P7.62mm_Horizontal, B.Cu at (405.9, 141.9)
- added D31: 1N4148, Diode_THT:D_DO-35_SOD27_P7.62mm_Horizontal, B.Cu at (425.0, 141.9)
- added D32: 1N4148, Diode_THT:D_DO-35_SOD27_P7.62mm_Horizontal, B.Cu at (444.0, 141.9)
- added D33: 1N4148, Diode_THT:D_DO-35_SOD27_P7.62mm_Horizontal, B.Cu at (467.9, 141.9)
- added D34: 1N4148, Diode_THT:D_DO-35_SOD27_P7.62mm_Horizontal, B.Cu at (486.9, 141.9)
- added D35: 1N4148, Diode_THT:D_DO-35_SOD27_P7.62mm_Horizontal, B.Cu at (506.0, 141.9)
- added D36: 1N4148, Diode_THT:D_DO-35_SOD27_P7.62mm_Horizontal, B.Cu at (525.0, 141.9)
- added D37: 1N4148, Diode_THT:D_DO-35_SOD27_P7.62mm_Horizontal, B.Cu at (120.2, 160.9)
- added D38: 1N4148, Diode_THT:D_DO-35_SOD27_P7.62mm_Horizontal, B.Cu at (144.0, 160.9)
- added D39: 1N4148, Diode_THT:D_DO-35_SOD27_P7.62mm_Horizontal, B.Cu at (163.1, 160.9)
- added D4: 1N4148, Diode_THT:D_DO-35_SOD27_P7.62mm_Horizontal, B.Cu at (210.7, 113.3)
- added D40: 1N4148, Diode_THT:D_DO-35_SOD27_P7.62mm_Horizontal, B.Cu at (182.1, 160.9)
- added D41: 1N4148, Diode_THT:D_DO-35_SOD27_P7.62mm_Horizontal, B.Cu at (201.2, 160.9)
- added D42: 1N4148, Diode_THT:D_DO-35_SOD27_P7.62mm_Horizontal, B.Cu at (220.2, 160.9)
- added D43: 1N4148, Diode_THT:D_DO-35_SOD27_P7.62mm_Horizontal, B.Cu at (239.3, 160.9)
- added D44: 1N4148, Diode_THT:D_DO-35_SOD27_P7.62mm_Horizontal, B.Cu at (258.3, 160.9)
- added D45: 1N4148, Diode_THT:D_DO-35_SOD27_P7.62mm_Horizontal, B.Cu at (277.4, 160.9)
- added D46: 1N4148, Diode_THT:D_DO-35_SOD27_P7.62mm_Horizontal, B.Cu at (296.4, 160.9)
- added D47: 1N4148, Diode_THT:D_DO-35_SOD27_P7.62mm_Horizontal, B.Cu at (315.5, 160.9)
- added D48: 1N4148, Diode_THT:D_DO-35_SOD27_P7.62mm_Horizontal, B.Cu at (334.5, 160.9)
- added D49: 1N4148, Diode_THT:D_DO-35_SOD27_P7.62mm_Horizontal, B.Cu at (353.6, 160.9)
- added D5: 1N4148, Diode_THT:D_DO-35_SOD27_P7.62mm_Horizontal, B.Cu at (239.3, 113.3)
- added D50: 1N4148, Diode_THT:D_DO-35_SOD27_P7.62mm_Horizontal, B.Cu at (377.4, 160.9)
- added D51: 1N4148, Diode_THT:D_DO-35_SOD27_P7.62mm_Horizontal, B.Cu at (405.9, 160.9)
- added D52: 1N4148, Diode_THT:D_DO-35_SOD27_P7.62mm_Horizontal, B.Cu at (425.0, 160.9)
- added D53: 1N4148, Diode_THT:D_DO-35_SOD27_P7.62mm_Horizontal, B.Cu at (444.0, 160.9)
- added D54: 1N4148, Diode_THT:D_DO-35_SOD27_P7.62mm_Horizontal, B.Cu at (467.9, 160.9)
- added D55: 1N4148, Diode_THT:D_DO-35_SOD27_P7.62mm_Horizontal, B.Cu at (486.9, 160.9)
- added D56: 1N4148, Diode_THT:D_DO-35_SOD27_P7.62mm_Horizontal, B.Cu at (506.0, 160.9)
- added D57: 1N4148, Diode_THT:D_DO-35_SOD27_P7.62mm_Horizontal, B.Cu at (525.0, 170.5)
- added D58: 1N4148, Diode_THT:D_DO-35_SOD27_P7.62mm_Horizontal, B.Cu at (122.6, 180.0)
- added D59: 1N4148, Diode_THT:D_DO-35_SOD27_P7.62mm_Horizontal, B.Cu at (148.8, 180.0)
- added D6: 1N4148, Diode_THT:D_DO-35_SOD27_P7.62mm_Horizontal, B.Cu at (258.3, 113.3)
- added D60: 1N4148, Diode_THT:D_DO-35_SOD27_P7.62mm_Horizontal, B.Cu at (167.8, 180.0)
- added D61: 1N4148, Diode_THT:D_DO-35_SOD27_P7.62mm_Horizontal, B.Cu at (186.9, 180.0)
- added D62: 1N4148, Diode_THT:D_DO-35_SOD27_P7.62mm_Horizontal, B.Cu at (205.9, 180.0)
- added D63: 1N4148, Diode_THT:D_DO-35_SOD27_P7.62mm_Horizontal, B.Cu at (225.0, 180.0)
- added D64: 1N4148, Diode_THT:D_DO-35_SOD27_P7.62mm_Horizontal, B.Cu at (244.0, 180.0)
- added D65: 1N4148, Diode_THT:D_DO-35_SOD27_P7.62mm_Horizontal, B.Cu at (263.1, 180.0)
- added D66: 1N4148, Diode_THT:D_DO-35_SOD27_P7.62mm_Horizontal, B.Cu at (282.1, 180.0)
- added D67: 1N4148, Diode_THT:D_DO-35_SOD27_P7.62mm_Horizontal, B.Cu at (301.2, 180.0)
- added D68: 1N4148, Diode_THT:D_DO-35_SOD27_P7.62mm_Horizontal, B.Cu at (320.2, 180.0)
- added D69: 1N4148, Diode_THT:D_DO-35_SOD27_P7.62mm_Horizontal, B.Cu at (339.3, 180.0)
- added D7: 1N4148, Diode_THT:D_DO-35_SOD27_P7.62mm_Horizontal, B.Cu at (277.4, 113.3)
- added D70: 1N4148, Diode_THT:D_DO-35_SOD27_P7.62mm_Horizontal, B.Cu at (370.2, 180.0)
- added D71: 1N4148, Diode_THT:D_DO-35_SOD27_P7.62mm_Horizontal, B.Cu at (467.9, 180.0)
- added D72: 1N4148, Diode_THT:D_DO-35_SOD27_P7.62mm_Horizontal, B.Cu at (486.9, 180.0)
- added D73: 1N4148, Diode_THT:D_DO-35_SOD27_P7.62mm_Horizontal, B.Cu at (506.0, 180.0)
- added D75: 1N4148, Diode_THT:D_DO-35_SOD27_P7.62mm_Horizontal, B.Cu at (127.3, 199.0)
- added D76: 1N4148, Diode_THT:D_DO-35_SOD27_P7.62mm_Horizontal, B.Cu at (158.3, 199.0)
- added D77: 1N4148, Diode_THT:D_DO-35_SOD27_P7.62mm_Horizontal, B.Cu at (177.3, 199.0)
- added D78: 1N4148, Diode_THT:D_DO-35_SOD27_P7.62mm_Horizontal, B.Cu at (196.4, 199.0)
- added D79: 1N4148, Diode_THT:D_DO-35_SOD27_P7.62mm_Horizontal, B.Cu at (215.4, 199.0)
- added D8: 1N4148, Diode_THT:D_DO-35_SOD27_P7.62mm_Horizontal, B.Cu at (296.4, 113.3)
- added D80: 1N4148, Diode_THT:D_DO-35_SOD27_P7.62mm_Horizontal, B.Cu at (234.5, 199.0)
- added D81: 1N4148, Diode_THT:D_DO-35_SOD27_P7.62mm_Horizontal, B.Cu at (253.5, 199.0)
- added D82: 1N4148, Diode_THT:D_DO-35_SOD27_P7.62mm_Horizontal, B.Cu at (272.6, 199.0)
- added D83: 1N4148, Diode_THT:D_DO-35_SOD27_P7.62mm_Horizontal, B.Cu at (291.6, 199.0)
- added D84: 1N4148, Diode_THT:D_DO-35_SOD27_P7.62mm_Horizontal, B.Cu at (310.7, 199.0)
- added D85: 1N4148, Diode_THT:D_DO-35_SOD27_P7.62mm_Horizontal, B.Cu at (329.7, 199.0)
- added D86: 1N4148, Diode_THT:D_DO-35_SOD27_P7.62mm_Horizontal, B.Cu at (365.5, 199.0)
- added D87: 1N4148, Diode_THT:D_DO-35_SOD27_P7.62mm_Horizontal, B.Cu at (425.0, 199.0)
- added D88: 1N4148, Diode_THT:D_DO-35_SOD27_P7.62mm_Horizontal, B.Cu at (467.9, 199.0)
- added D89: 1N4148, Diode_THT:D_DO-35_SOD27_P7.62mm_Horizontal, B.Cu at (486.9, 199.0)
- added D9: 1N4148, Diode_THT:D_DO-35_SOD27_P7.62mm_Horizontal, B.Cu at (325.0, 113.3)
- added D90: 1N4148, Diode_THT:D_DO-35_SOD27_P7.62mm_Horizontal, B.Cu at (506.0, 199.0)
- added D91: 1N4148, Diode_THT:D_DO-35_SOD27_P7.62mm_Horizontal, B.Cu at (525.0, 208.6)
- added D92: 1N4148, Diode_THT:D_DO-35_SOD27_P7.62mm_Horizontal, B.Cu at (117.8, 218.1)
- added D93: 1N4148, Diode_THT:D_DO-35_SOD27_P7.62mm_Horizontal, B.Cu at (141.6, 218.1)
- added D94: 1N4148, Diode_THT:D_DO-35_SOD27_P7.62mm_Horizontal, B.Cu at (165.4, 218.1)
- added D95: 1N4148, Diode_THT:D_DO-35_SOD27_P7.62mm_Horizontal, B.Cu at (236.9, 218.1)
- added D96: 1N4148, Diode_THT:D_DO-35_SOD27_P7.62mm_Horizontal, B.Cu at (308.3, 218.1)
- added D97: 1N4148, Diode_THT:D_DO-35_SOD27_P7.62mm_Horizontal, B.Cu at (332.1, 218.1)
- added D98: 1N4148, Diode_THT:D_DO-35_SOD27_P7.62mm_Horizontal, B.Cu at (355.9, 218.1)
- added D99: 1N4148, Diode_THT:D_DO-35_SOD27_P7.62mm_Horizontal, B.Cu at (379.7, 218.1)
- added S1: MX_stab, PCM_marbastlib-mx:STAB_MX_2u, F.Cu at (367.5, 137.9)
- added S2: MX_stab, PCM_marbastlib-mx:STAB_MX_2u, F.Cu at (519.9, 166.5)
- added S3: MX_stab, PCM_marbastlib-mx:STAB_MX_2u, F.Cu at (519.9, 204.6)
- added S4: MX_stab, PCM_marbastlib-mx:STAB_MX_2u, F.Cu at (472.3, 214.1)
- added S5: MX_stab, PCM_marbastlib-mx:STAB_MX_2.25u, F.Cu at (122.3, 195.0)
- added S5: MX_stab, PCM_marbastlib-mx:STAB_MX_2.25u, F.Cu at (365.1, 176.0)
- added S6: MX_stab, PCM_marbastlib-mx:STAB_MX_2.75u, F.Cu at (360.4, 195.0)
- added S7: MX_stab, PCM_marbastlib-mx:STAB_MX_6.25u, F.Cu at (231.8, 214.1)
- added SW1: RotaryEncoder_Switch, Rotary_Encoder:RotaryEncoder_Alps_EC11E-Switch_Vertical_H20mm, F.Cu at (110.2, 106.7)
- added SW10: SW_Push, PCM_marbastlib-mx:SW_MX_HS_CPG151101S11_1u, F.Cu at (319.9, 109.3)
- added SW100: SW_Push, PCM_marbastlib-mx:SW_MX_HS_CPG151101S11_1u, F.Cu at (374.7, 214.1)
- added SW101: SW_Push, PCM_marbastlib-mx:SW_MX_HS_CPG151101S11_1u, F.Cu at (400.9, 214.1)
- added SW102: SW_Push, PCM_marbastlib-mx:SW_MX_HS_CPG151101S11_1u, F.Cu at (419.9, 214.1)
- added SW103: SW_Push, PCM_marbastlib-mx:SW_MX_HS_CPG151101S11_1u, F.Cu at (439.0, 214.1)
- added SW104: SW_Push, PCM_marbastlib-mx:SW_MX_HS_CPG151101S11_1u, F.Cu at (472.3, 214.1)
- added SW105: SW_Push, PCM_marbastlib-mx:SW_MX_HS_CPG151101S11_1u, F.Cu at (500.9, 214.1)
- added SW11: SW_Push, PCM_marbastlib-mx:SW_MX_HS_CPG151101S11_1u, F.Cu at (338.9, 109.3)
- added SW12: SW_Push, PCM_marbastlib-mx:SW_MX_HS_CPG151101S11_1u, F.Cu at (358.0, 109.3)
- added SW13: SW_Push, PCM_marbastlib-mx:SW_MX_HS_CPG151101S11_1u, F.Cu at (377.0, 109.3)
- added SW14: SW_Push, PCM_marbastlib-mx:SW_MX_HS_CPG151101S11_1u, F.Cu at (400.9, 109.3)
- added SW15: SW_Push, PCM_marbastlib-mx:SW_MX_HS_CPG151101S11_1u, F.Cu at (419.9, 109.3)
- added SW16: SW_Push, PCM_marbastlib-mx:SW_MX_HS_CPG151101S11_1u, F.Cu at (439.0, 109.3)
- added SW17: SW_Push, PCM_marbastlib-mx:SW_MX_HS_CPG151101S11_1u, F.Cu at (110.3, 137.9)
- added SW18: SW_Push, PCM_marbastlib-mx:SW_MX_HS_CPG151101S11_1u, F.Cu at (129.4, 137.9)
- added SW19: SW_Push, PCM_marbastlib-mx:SW_MX_HS_CPG151101S11_1u, F.Cu at (148.4, 137.9)
- added SW2: SW_Push, PCM_marbastlib-mx:SW_MX_HS_CPG151101S11_1u, F.Cu at (148.4, 109.3)
- added SW20: SW_Push, PCM_marbastlib-mx:SW_MX_HS_CPG151101S11_1u, F.Cu at (167.5, 137.9)
- added SW21: SW_Push, PCM_marbastlib-mx:SW_MX_HS_CPG151101S11_1u, F.Cu at (186.5, 137.9)
- added SW22: SW_Push, PCM_marbastlib-mx:SW_MX_HS_CPG151101S11_1u, F.Cu at (205.6, 137.9)
- added SW23: SW_Push, PCM_marbastlib-mx:SW_MX_HS_CPG151101S11_1u, F.Cu at (224.6, 137.9)
- added SW24: SW_Push, PCM_marbastlib-mx:SW_MX_HS_CPG151101S11_1u, F.Cu at (243.7, 137.9)
- added SW25: SW_Push, PCM_marbastlib-mx:SW_MX_HS_CPG151101S11_1u, F.Cu at (262.7, 137.9)
- added SW26: SW_Push, PCM_marbastlib-mx:SW_MX_HS_CPG151101S11_1u, F.Cu at (281.8, 137.9)
- added SW27: SW_Push, PCM_marbastlib-mx:SW_MX_HS_CPG151101S11_1u, F.Cu at (300.8, 137.9)
- added SW28: SW_Push, PCM_marbastlib-mx:SW_MX_HS_CPG151101S11_1u, F.Cu at (319.9, 137.9)
- added SW29: SW_Push, PCM_marbastlib-mx:SW_MX_HS_CPG151101S11_1u, F.Cu at (338.9, 137.9)
- added SW3: SW_Push, PCM_marbastlib-mx:SW_MX_HS_CPG151101S11_1u, F.Cu at (167.5, 109.3)
- added SW30: SW_Push, PCM_marbastlib-mx:SW_MX_HS_CPG151101S11_1u, F.Cu at (367.5, 137.9)
- added SW31: SW_Push, PCM_marbastlib-mx:SW_MX_HS_CPG151101S11_1u, F.Cu at (400.9, 137.9)
- added SW32: SW_Push, PCM_marbastlib-mx:SW_MX_HS_CPG151101S11_1u, F.Cu at (419.9, 137.9)
- added SW33: SW_Push, PCM_marbastlib-mx:SW_MX_HS_CPG151101S11_1u, F.Cu at (439.0, 137.9)
- added SW34: SW_Push, PCM_marbastlib-mx:SW_MX_HS_CPG151101S11_1u, F.Cu at (462.8, 137.9)
- added SW35: SW_Push, PCM_marbastlib-mx:SW_MX_HS_CPG151101S11_1u, F.Cu at (481.8, 137.9)
- added SW36: SW_Push, PCM_marbastlib-mx:SW_MX_HS_CPG151101S11_1u, F.Cu at (500.9, 137.9)
- added SW37: SW_Push, PCM_marbastlib-mx:SW_MX_HS_CPG151101S11_1u, F.Cu at (519.9, 137.9)
- added SW38: SW_Push, PCM_marbastlib-mx:SW_MX_HS_CPG151101S11_1u, F.Cu at (115.1, 156.9)
- added SW39: SW_Push, PCM_marbastlib-mx:SW_MX_HS_CPG151101S11_1u, F.Cu at (138.9, 156.9)
- added SW4: SW_Push, PCM_marbastlib-mx:SW_MX_HS_CPG151101S11_1u, F.Cu at (186.5, 109.3)
- added SW40: SW_Push, PCM_marbastlib-mx:SW_MX_HS_CPG151101S11_1u, F.Cu at (158.0, 156.9)
- added SW41: SW_Push, PCM_marbastlib-mx:SW_MX_HS_CPG151101S11_1u, F.Cu at (177.0, 156.9)
- added SW42: SW_Push, PCM_marbastlib-mx:SW_MX_HS_CPG151101S11_1u, F.Cu at (196.1, 156.9)
- added SW43: SW_Push, PCM_marbastlib-mx:SW_MX_HS_CPG151101S11_1u, F.Cu at (215.1, 156.9)
- added SW44: SW_Push, PCM_marbastlib-mx:SW_MX_HS_CPG151101S11_1u, F.Cu at (234.2, 156.9)
- added SW45: SW_Push, PCM_marbastlib-mx:SW_MX_HS_CPG151101S11_1u, F.Cu at (253.2, 156.9)
- added SW46: SW_Push, PCM_marbastlib-mx:SW_MX_HS_CPG151101S11_1u, F.Cu at (272.3, 156.9)
- added SW47: SW_Push, PCM_marbastlib-mx:SW_MX_HS_CPG151101S11_1u, F.Cu at (291.3, 156.9)
- added SW48: SW_Push, PCM_marbastlib-mx:SW_MX_HS_CPG151101S11_1u, F.Cu at (310.4, 156.9)
- added SW49: SW_Push, PCM_marbastlib-mx:SW_MX_HS_CPG151101S11_1u, F.Cu at (329.4, 156.9)
- added SW5: SW_Push, PCM_marbastlib-mx:SW_MX_HS_CPG151101S11_1u, F.Cu at (205.6, 109.3)
- added SW50: SW_Push, PCM_marbastlib-mx:SW_MX_HS_CPG151101S11_1u, F.Cu at (348.5, 156.9)
- added SW51: SW_Push, PCM_marbastlib-mx:SW_MX_HS_CPG151101S11_1u, F.Cu at (372.3, 156.9)
- added SW52: SW_Push, PCM_marbastlib-mx:SW_MX_HS_CPG151101S11_1u, F.Cu at (400.9, 156.9)
- added SW53: SW_Push, PCM_marbastlib-mx:SW_MX_HS_CPG151101S11_1u, F.Cu at (419.9, 156.9)
- added SW54: SW_Push, PCM_marbastlib-mx:SW_MX_HS_CPG151101S11_1u, F.Cu at (439.0, 156.9)
- added SW55: SW_Push, PCM_marbastlib-mx:SW_MX_HS_CPG151101S11_1u, F.Cu at (462.8, 156.9)
- added SW56: SW_Push, PCM_marbastlib-mx:SW_MX_HS_CPG151101S11_1u, F.Cu at (481.8, 156.9)
- added SW57: SW_Push, PCM_marbastlib-mx:SW_MX_HS_CPG151101S11_1u, F.Cu at (500.9, 156.9)
- added SW58: SW_Push, PCM_marbastlib-mx:SW_MX_HS_CPG151101S11_1u, F.Cu at (519.9, 166.5)
- added SW59: SW_Push, PCM_marbastlib-mx:SW_MX_HS_CPG151101S11_1u, F.Cu at (117.5, 176.0)
- added SW6: SW_Push, PCM_marbastlib-mx:SW_MX_HS_CPG151101S11_1u, F.Cu at (234.2, 109.3)
- added SW60: SW_Push, PCM_marbastlib-mx:SW_MX_HS_CPG151101S11_1u, F.Cu at (143.7, 176.0)
- added SW61: SW_Push, PCM_marbastlib-mx:SW_MX_HS_CPG151101S11_1u, F.Cu at (162.7, 176.0)
- added SW62: SW_Push, PCM_marbastlib-mx:SW_MX_HS_CPG151101S11_1u, F.Cu at (181.8, 176.0)
- added SW63: SW_Push, PCM_marbastlib-mx:SW_MX_HS_CPG151101S11_1u, F.Cu at (200.8, 176.0)
- added SW64: SW_Push, PCM_marbastlib-mx:SW_MX_HS_CPG151101S11_1u, F.Cu at (219.9, 176.0)
- added SW65: SW_Push, PCM_marbastlib-mx:SW_MX_HS_CPG151101S11_1u, F.Cu at (238.9, 176.0)
- added SW66: SW_Push, PCM_marbastlib-mx:SW_MX_HS_CPG151101S11_1u, F.Cu at (258.0, 176.0)
- added SW67: SW_Push, PCM_marbastlib-mx:SW_MX_HS_CPG151101S11_1u, F.Cu at (277.0, 176.0)
- added SW68: SW_Push, PCM_marbastlib-mx:SW_MX_HS_CPG151101S11_1u, F.Cu at (296.1, 176.0)
- added SW69: SW_Push, PCM_marbastlib-mx:SW_MX_HS_CPG151101S11_1u, F.Cu at (315.1, 176.0)
- added SW7: SW_Push, PCM_marbastlib-mx:SW_MX_HS_CPG151101S11_1u, F.Cu at (253.2, 109.3)
- added SW70: SW_Push, PCM_marbastlib-mx:SW_MX_HS_CPG151101S11_1u, F.Cu at (334.2, 176.0)
- added SW71: SW_Push, PCM_marbastlib-mx:SW_MX_HS_CPG151101S11_1u, F.Cu at (365.1, 176.0)
- added SW72: SW_Push, PCM_marbastlib-mx:SW_MX_HS_CPG151101S11_1u, F.Cu at (462.8, 176.0)
- added SW73: SW_Push, PCM_marbastlib-mx:SW_MX_HS_CPG151101S11_1u, F.Cu at (481.8, 176.0)
- added SW74: SW_Push, PCM_marbastlib-mx:SW_MX_HS_CPG151101S11_1u, F.Cu at (500.9, 176.0)
- added SW76: SW_Push, PCM_marbastlib-mx:SW_MX_HS_CPG151101S11_1u, F.Cu at (122.3, 195.0)
- added SW77: SW_Push, PCM_marbastlib-mx:SW_MX_HS_CPG151101S11_1u, F.Cu at (153.2, 195.0)
- added SW78: SW_Push, PCM_marbastlib-mx:SW_MX_HS_CPG151101S11_1u, F.Cu at (172.3, 195.0)
- added SW79: SW_Push, PCM_marbastlib-mx:SW_MX_HS_CPG151101S11_1u, F.Cu at (191.3, 195.0)
- added SW8: SW_Push, PCM_marbastlib-mx:SW_MX_HS_CPG151101S11_1u, F.Cu at (272.3, 109.3)
- added SW80: SW_Push, PCM_marbastlib-mx:SW_MX_HS_CPG151101S11_1u, F.Cu at (210.4, 195.0)
- added SW81: SW_Push, PCM_marbastlib-mx:SW_MX_HS_CPG151101S11_1u, F.Cu at (229.4, 195.0)
- added SW82: SW_Push, PCM_marbastlib-mx:SW_MX_HS_CPG151101S11_1u, F.Cu at (248.5, 195.0)
- added SW83: SW_Push, PCM_marbastlib-mx:SW_MX_HS_CPG151101S11_1u, F.Cu at (267.5, 195.0)
- added SW84: SW_Push, PCM_marbastlib-mx:SW_MX_HS_CPG151101S11_1u, F.Cu at (286.6, 195.0)
- added SW85: SW_Push, PCM_marbastlib-mx:SW_MX_HS_CPG151101S11_1u, F.Cu at (305.6, 195.0)
- added SW86: SW_Push, PCM_marbastlib-mx:SW_MX_HS_CPG151101S11_1u, F.Cu at (324.7, 195.0)
- added SW87: SW_Push, PCM_marbastlib-mx:SW_MX_HS_CPG151101S11_1u, F.Cu at (360.4, 195.0)
- added SW88: SW_Push, PCM_marbastlib-mx:SW_MX_HS_CPG151101S11_1.25u, F.Cu at (419.9, 195.0)
- added SW89: SW_Push, PCM_marbastlib-mx:SW_MX_HS_CPG151101S11_1u, F.Cu at (462.8, 195.0)
- added SW9: SW_Push, PCM_marbastlib-mx:SW_MX_HS_CPG151101S11_1u, F.Cu at (291.3, 109.3)
- added SW90: SW_Push, PCM_marbastlib-mx:SW_MX_HS_CPG151101S11_1u, F.Cu at (481.8, 195.0)
- added SW91: SW_Push, PCM_marbastlib-mx:SW_MX_HS_CPG151101S11_1u, F.Cu at (500.9, 195.0)
- added SW92: SW_Push, PCM_marbastlib-mx:SW_MX_HS_CPG151101S11_1u, F.Cu at (519.9, 204.6)
- added SW93: SW_Push, PCM_marbastlib-mx:SW_MX_HS_CPG151101S11_1.25u, F.Cu at (112.7, 214.1)
- added SW94: SW_Push, PCM_marbastlib-mx:SW_MX_HS_CPG151101S11_1u, F.Cu at (136.5, 214.1)
- added SW95: SW_Push, PCM_marbastlib-mx:SW_MX_HS_CPG151101S11_1u, F.Cu at (160.4, 214.1)
- added SW96: SW_Push, PCM_marbastlib-mx:SW_MX_HS_CPG151101S11_1u, F.Cu at (231.8, 214.1)
- added SW97: SW_Push, PCM_marbastlib-mx:SW_MX_HS_CPG151101S11_1u, F.Cu at (303.2, 214.1)
- added SW98: SW_Push, PCM_marbastlib-mx:SW_MX_HS_CPG151101S11_1u, F.Cu at (327.0, 214.1)
- added SW99: SW_Push, PCM_marbastlib-mx:SW_MX_HS_CPG151101S11_1u, F.Cu at (350.9, 214.1)
- added U1: ESP32-S3-DevKitC, PCM_Espressif:ESP32-S3-DevKitC, F.Cu at (89.0, 167.5)
Other:
- board outline added: 502.4 x 209.1 mm

Commit message: Finishing up the pcb
did all routing, wiring, etc...
Parts:
- removed the D1 at (153.5, 113.3)
- removed the S5 at (122.3, 195.0)
- removed the S5 at (365.1, 176.0)
- removed the SW2 at (148.4, 109.3)
- added D1: 1N4148, Diode_SMD:D_SOD-123, B.Cu at (150.5, 84.0)
- added D1: 1N4148, Diode_SMD:D_SOD-123, B.Cu at (112.2, 84.0)
- added S5: MX_stab, PCM_marbastlib-mx:STAB_MX_2.25u, F.Cu at (118.9, 164.5)
- added S8: MX_stab, PCM_marbastlib-mx:STAB_MX_2.25u, F.Cu at (361.8, 145.5)
- added SW2: SW_Push, PCM_marbastlib-mx:SW_MX_HS_CPG151101S11_1u, B.Cu at (107.0, 78.8)
- added SW2: SW_Push, PCM_marbastlib-mx:SW_MX_HS_CPG151101S11_1u, B.Cu at (145.1, 78.8)
- D10, D100, D101, D102, D103, D104, D11, D12, D13, D14, D15, D16, D17, D18, D19, D2, D20, D21, D22, D23, D24, D25, D26, D27, D28, D29, D3, D30, D31, D32, D33, D34, D35, D36, D37, D38, D39, D4, D40, D41, D42, D43, D44, D45, D46, D47, D48, D49, D5, D50, D51, D52, D53, D54, D55, D56, D57, D58, D59, D6, D60, D61, D62, D63, D64, D65, D66, D67, D68, D69, D7, D70, D71, D72, D73, D75, D76, D77, D78, D79, D8, D80, D81, D82, D83, D84, D85, D86, D87, D88, D89, D9, D90, D91, D92, D93, D94, D95, D96, D97, D98, D99: footprint Diode_THT:D_DO-35_SOD27_P7.62mm_Horizontal -> Diode_SMD:D_SOD-123
- SW10, SW100, SW101, SW102, SW105, SW11, SW12, SW13, SW14, SW15, SW16, SW17, SW18, SW19, SW20, SW21, SW22, SW23, SW24, SW25, SW26, SW27, SW28, SW29, SW3, SW30, SW31, SW32, SW33, SW34, SW35, SW36, SW37, SW38, SW39, SW4, SW40, SW41, SW42, SW43, SW44, SW45, SW46, SW47, SW48, SW49, SW5, SW50, SW51, SW52, SW53, SW54, SW55, SW56, SW57, SW58, SW59, SW6, SW60, SW61, SW62, SW63, SW64, SW65, SW66, SW67, SW68, SW69, SW7, SW70, SW71, SW72, SW73, SW74, SW76, SW77, SW78, SW79, SW8, SW80, SW81, SW82, SW83, SW84, SW85, SW86, SW87, SW89, SW9, SW90, SW91, SW92, SW93, SW95, SW96, SW97, SW98, SW99: moved to B.Cu
- SW103, SW104, SW94: footprint PCM_marbastlib-mx:SW_MX_HS_CPG151101S11_1u -> PCM_marbastlib-mx:SW_MX_HS_CPG151101S11_1.25u; moved to B.Cu
- SW88: footprint PCM_marbastlib-mx:SW_MX_HS_CPG151101S11_1.25u -> PCM_marbastlib-mx:SW_MX_HS_CPG151101S11_1u; moved to B.Cu
- moved SW1 381.0 mm to (490.0, 76.0)
- moved S3 183.6 mm to (364.1, 107.4), turned to 0 degrees
- moved S1 149.0 mm to (516.5, 136.0), turned to 90 degrees
- moved S4 59.7 mm to (516.5, 174.1), turned to 90 degrees
- moved S2 53.8 mm to (468.9, 183.6), turned to 0 degrees
- moved U1 42.0 mm to (87.0, 125.5)
- moved SW100 30.7 mm to (371.3, 183.6), turned to 180 degrees
- moved SW11 30.7 mm to (335.6, 78.8), turned to 180 degrees
- moved SW20 30.7 mm to (164.1, 107.4), turned to 180 degrees
- moved SW23 30.7 mm to (221.3, 107.4), turned to 180 degrees
- moved SW29 30.7 mm to (335.6, 107.4), turned to 180 degrees
- moved SW3 30.7 mm to (164.1, 78.8), turned to 180 degrees
- moved SW35 30.7 mm to (478.4, 107.4), turned to 180 degrees
- moved SW41 30.7 mm to (173.6, 126.4), turned to 180 degrees
- moved SW43 30.7 mm to (211.7, 126.4), turned to 180 degrees
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Connections:
- D10 pad 1: /ROW5 -> (no net)
- D10 pad 2: Net-(D10-A) -> (no net)
- D100 pad 1: /ROW4 -> (no net)
- D100 pad 2: Net-(D100-A) -> (no net)
- D101 pad 1: /ROW5 -> (no net)
- D101 pad 2: Net-(D101-A) -> (no net)
- D102 pad 1: /ROW1 -> (no net)
- D102 pad 2: Net-(D102-A) -> (no net)
- D103 pad 1: /ROW2 -> (no net)
- D103 pad 2: Net-(D103-A) -> (no net)
- D104 pad 1: /ROW4 -> (no net)
- D104 pad 2: Net-(D104-A) -> (no net)
- D11 pad 1: /ROW0 -> (no net)
- D11 pad 2: Net-(D11-A) -> (no net)
- D12 pad 1: /ROW1 -> (no net)
- D12 pad 2: Net-(D12-A) -> (no net)
- D13 pad 1: /ROW2 -> (no net)
- D13 pad 2: Net-(D13-A) -> (no net)
- D14 pad 1: /ROW3 -> (no net)
- D14 pad 2: Net-(D14-A) -> (no net)
- D15 pad 1: /ROW4 -> (no net)
- D15 pad 2: Net-(D15-A) -> (no net)
- D16 pad 1: /ROW5 -> (no net)
- D16 pad 2: Net-(D16-A) -> (no net)
- D17 pad 1: /ROW0 -> (no net)
- D17 pad 2: Net-(D17-A) -> (no net)
- D18 pad 1: /ROW1 -> (no net)
- D18 pad 2: Net-(D18-A) -> (no net)
- D19 pad 1: /ROW2 -> (no net)
- D19 pad 2: Net-(D19-A) -> (no net)
- D2 pad 1: /ROW1 -> (no net)
- D2 pad 2: Net-(D2-A) -> (no net)
- D20 pad 1: /ROW3 -> (no net)
- D20 pad 2: Net-(D20-A) -> (no net)
- D21 pad 1: /ROW4 -> (no net)
- D21 pad 2: Net-(D21-A) -> (no net)
- D22 pad 1: /ROW0 -> (no net)
- D22 pad 2: Net-(D22-A) -> (no net)
- D23 pad 1: /ROW1 -> (no net)
- D23 pad 2: Net-(D23-A) -> (no net)
- D24 pad 1: /ROW2 -> (no net)
- D24 pad 2: Net-(D24-A) -> (no net)
- D25 pad 1: /ROW3 -> (no net)
- D25 pad 2: Net-(D25-A) -> (no net)
- D26 pad 1: /ROW4 -> (no net)
- D26 pad 2: Net-(D26-A) -> (no net)
- D27 pad 1: /ROW0 -> (no net)
- D27 pad 2: Net-(D27-A) -> (no net)
- D28 pad 1: /ROW1 -> (no net)
- D28 pad 2: Net-(D28-A) -> (no net)
- D29 pad 1: /ROW2 -> (no net)
- D29 pad 2: Net-(D29-A) -> (no net)
- D3 pad 1: /ROW2 -> (no net)
- D3 pad 2: Net-(D3-A) -> (no net)
- D30 pad 1: /ROW3 -> (no net)
- D30 pad 2: Net-(D30-A) -> (no net)
- D31 pad 1: /ROW4 -> (no net)
- D31 pad 2: Net-(D31-A) -> (no net)
- D32 pad 1: /ROW5 -> (no net)
- D32 pad 2: Net-(D32-A) -> (no net)
- D33 pad 1: /ROW0 -> (no net)
- D33 pad 2: Net-(D33-A) -> (no net)
- D34 pad 1: /ROW1 -> (no net)
- D34 pad 2: Net-(D34-A) -> (no net)
- D35 pad 1: /ROW2 -> (no net)
- D35 pad 2: Net-(D35-A) -> (no net)
- D36 pad 1: /ROW3 -> (no net)
- D36 pad 2: Net-(D36-A) -> (no net)
- D37 pad 1: /ROW4 -> (no net)
- D37 pad 2: Net-(D37-A) -> (no net)
- D38 pad 1: /ROW0 -> (no net)
- D38 pad 2: Net-(D38-A) -> (no net)
- D39 pad 1: /ROW1 -> (no net)
- D39 pad 2: Net-(D39-A) -> (no net)
- D4 pad 1: /ROW3 -> (no net)
- D4 pad 2: Net-(D4-A) -> (no net)
- D40 pad 1: /ROW2 -> (no net)
- D40 pad 2: Net-(D40-A) -> (no net)
- D41 pad 1: /ROW3 -> (no net)
- D41 pad 2: Net-(D41-A) -> (no net)
- D42 pad 1: /ROW4 -> (no net)
- D42 pad 2: Net-(D42-A) -> (no net)
- D43 pad 1: /ROW0 -> (no net)
- D43 pad 2: Net-(D43-A) -> (no net)
- D44 pad 1: /ROW1 -> (no net)
- D44 pad 2: Net-(D44-A) -> (no net)
- D45 pad 1: /ROW2 -> (no net)
- D45 pad 2: Net-(D45-A) -> (no net)
- D46 pad 1: /ROW3 -> (no net)
- D46 pad 2: Net-(D46-A) -> (no net)
- D47 pad 1: /ROW4 -> (no net)
- D47 pad 2: Net-(D47-A) -> (no net)
- D48 pad 1: /ROW0 -> (no net)
- D48 pad 2: Net-(D48-A) -> (no net)
- D49 pad 1: /ROW1 -> (no net)
- D49 pad 2: Net-(D49-A) -> (no net)
- D5 pad 1: /ROW5 -> (no net)
- D5 pad 2: Net-(D5-A) -> (no net)
- D50 pad 1: /ROW2 -> (no net)
- D50 pad 2: Net-(D50-A) -> (no net)
- D51 pad 1: /ROW3 -> (no net)
- D51 pad 2: Net-(D51-A) -> (no net)
- D52 pad 1: /ROW4 -> (no net)
- D52 pad 2: Net-(D52-A) -> (no net)
- D53 pad 1: /ROW0 -> (no net)
- D53 pad 2: Net-(D53-A) -> (no net)
- D54 pad 1: /ROW1 -> (no net)
- D54 pad 2: Net-(D54-A) -> (no net)
- D55 pad 1: /ROW2 -> (no net)
- D55 pad 2: Net-(D55-A) -> (no net)
- D56 pad 1: /ROW3 -> (no net)
- D56 pad 2: Net-(D56-A) -> (no net)
- D57 pad 1: /ROW4 -> (no net)
- D57 pad 2: Net-(D57-A) -> (no net)
- D58 pad 1: /ROW5 -> (no net)
- D58 pad 2: Net-(D58-A) -> (no net)
- D59 pad 1: /ROW0 -> (no net)
- D59 pad 2: Net-(D59-A) -> (no net)
- D6 pad 1: /ROW1 -> (no net)
- D6 pad 2: Net-(D6-A) -> (no net)
- D60 pad 1: /ROW1 -> (no net)
- D60 pad 2: Net-(D60-A) -> (no net)
- D61 pad 1: /ROW2 -> (no net)
- D61 pad 2: Net-(D61-A) -> (no net)
- D62 pad 1: /ROW3 -> (no net)
- D62 pad 2: Net-(D62-A) -> (no net)
- D63 pad 1: /ROW4 -> (no net)
- D63 pad 2: Net-(D63-A) -> (no net)
- D64 pad 1: /ROW5 -> (no net)
- D64 pad 2: Net-(D64-A) -> (no net)
- D65 pad 1: /ROW0 -> (no net)
- D65 pad 2: Net-(D65-A) -> (no net)
- D66 pad 1: /ROW1 -> (no net)
- D66 pad 2: Net-(D66-A) -> (no net)
- D67 pad 1: /ROW2 -> (no net)
- D67 pad 2: Net-(D67-A) -> (no net)
- D68 pad 1: /ROW3 -> (no net)
- D68 pad 2: Net-(D68-A) -> (no net)
- D69 pad 1: /ROW4 -> (no net)
- D69 pad 2: Net-(D69-A) -> (no net)
- D7 pad 1: /ROW2 -> (no net)
- D7 pad 2: Net-(D7-A) -> (no net)
- D70 pad 1: /ROW5 -> (no net)
- D70 pad 2: Net-(D70-A) -> (no net)
- D71 pad 1: /ROW0 -> (no net)
- D71 pad 2: Net-(D71-A) -> (no net)
- D72 pad 1: /ROW1 -> (no net)
- D72 pad 2: Net-(D72-A) -> (no net)
- D73 pad 1: /ROW2 -> (no net)
- D73 pad 2: Net-(D73-A) -> (no net)
- D75 pad 1: /ROW0 -> (no net)
- D75 pad 2: Net-(D75-A) -> (no net)
- D76 pad 1: /ROW1 -> (no net)
- D76 pad 2: Net-(D76-A) -> (no net)
- D77 pad 1: /ROW2 -> (no net)
- D77 pad 2: Net-(D77-A) -> (no net)
- D78 pad 1: /ROW5 -> (no net)
- D78 pad 2: Net-(D78-A) -> (no net)
- D79 pad 1: /ROW0 -> (no net)
- D79 pad 2: Net-(D79-A) -> (no net)
- D8 pad 1: /ROW3 -> (no net)
- D8 pad 2: Net-(D8-A) -> (no net)
- D80 pad 1: /ROW1 -> (no net)
- D80 pad 2: Net-(D80-A) -> (no net)
- D81 pad 1: /ROW2 -> (no net)
- D81 pad 2: Net-(D81-A) -> (no net)
- D82 pad 1: /ROW4 -> (no net)
- D82 pad 2: Net-(D82-A) -> (no net)
- D83 pad 1: /ROW5 -> (no net)
- D83 pad 2: Net-(D83-A) -> (no net)
- D84 pad 1: /ROW0 -> (no net)
- D84 pad 2: Net-(D84-A) -> (no net)
- D85 pad 1: /ROW1 -> (no net)
- D85 pad 2: Net-(D85-A) -> (no net)
- D86 pad 1: /ROW2 -> (no net)
- D86 pad 2: Net-(D86-A) -> (no net)
- D87 pad 1: /ROW5 -> (no net)
- D87 pad 2: Net-(D87-A) -> (no net)
- D88 pad 1: /ROW1 -> (no net)
- D88 pad 2: Net-(D88-A) -> (no net)
- D89 pad 1: /ROW2 -> (no net)
- D89 pad 2: Net-(D89-A) -> (no net)
- D9 pad 1: /ROW4 -> (no net)
- D9 pad 2: Net-(D9-A) -> (no net)
- D90 pad 1: /ROW3 -> (no net)
- D90 pad 2: Net-(D90-A) -> (no net)
- D91 pad 1: /ROW4 -> (no net)
- D91 pad 2: Net-(D91-A) -> (no net)
- D92 pad 1: /ROW5 -> (no net)
- D92 pad 2: Net-(D92-A) -> (no net)
- D93 pad 1: /ROW1 -> (no net)
- D93 pad 2: Net-(D93-A) -> (no net)
- D94 pad 1: /ROW2 -> (no net)
- D94 pad 2: Net-(D94-A) -> (no net)
- D95 pad 1: /ROW3 -> (no net)
- D95 pad 2: Net-(D95-A) -> (no net)
- D96 pad 1: /ROW4 -> (no net)
- D96 pad 2: Net-(D96-A) -> (no net)
- D97 pad 1: /ROW1 -> (no net)
- D97 pad 2: Net-(D97-A) -> (no net)
- D98 pad 1: /ROW2 -> (no net)
- D98 pad 2: Net-(D98-A) -> (no net)
- D99 pad 1: /ROW3 -> (no net)
- D99 pad 2: Net-(D99-A) -> (no net)
- SW10 pad 1: /COL1 -> /COL9
- SW100 pad 1: /COL19 -> /COL13
- SW101 pad 1: /COL19 -> /COL14
- SW102 pad 1: /COL19 -> /COL15
- SW103 pad 1: /COL20 -> /COL16
- SW104 pad 1: /COL20 -> /COL17
- SW105 pad 1: /COL20 -> /COL19
- SW11 pad 1: /COL1 -> /COL10
- SW12 pad 1: /COL2 -> /COL11
- SW13 pad 1: /COL2 -> /COL12
- SW14 pad 1: /COL2 -> /COL13
- SW15 pad 1: /COL2 -> /COL14
- SW16 pad 1: /COL2 -> /COL15
- SW17 pad 1: /COL2 -> /COL16
- SW18 pad 1: /COL3 -> (no net)
- SW18 pad 2: Net-(D17-A) -> (no net)
- SW19 pad 1: /COL3 -> /COL1
- SW20 pad 1: /COL3 -> /COL2
- SW22 pad 1: /COL3 -> /COL4
- SW23 pad 1: /COL4 -> /COL5
- SW24 pad 1: /COL4 -> /COL6
- SW25 pad 1: /COL4 -> /COL7
- SW26 pad 1: /COL4 -> /COL8
- SW27 pad 1: /COL4 -> /COL9
- SW28 pad 1: /COL5 -> /COL10
- SW29 pad 1: /COL5 -> /COL11
- SW3 pad 1: /COL0 -> /COL2
- SW30 pad 1: /COL5 -> /COL12
- SW31 pad 1: /COL5 -> /COL13
- SW32 pad 1: /COL5 -> /COL14
- SW33 pad 1: /COL5 -> /COL15
- SW34 pad 1: /COL6 -> /COL16
- SW35 pad 1: /COL6 -> /COL17
- SW36 pad 1: /COL6 -> /COL18
- SW37 pad 1: /COL6 -> /COL19
- SW38 pad 1: /COL6 -> /COL20
- SW39 pad 1: /COL7 -> (no net)
- SW39 pad 2: Net-(D38-A) -> (no net)
- SW4 pad 1: /COL0 -> /COL3
- SW40 pad 1: /COL7 -> /COL1
- SW41 pad 1: /COL7 -> /COL2
- SW42 pad 1: /COL7 -> /COL3
- SW43 pad 1: /COL7 -> /COL4
- SW44 pad 1: /COL8 -> /COL5
- SW45 pad 1: /COL8 -> /COL6
- SW46 pad 1: /COL8 -> /COL7
- SW48 pad 1: /COL8 -> /COL9
- SW49 pad 1: /COL9 -> /COL10
- SW5 pad 1: /COL0 -> /COL4
- SW50 pad 1: /COL9 -> /COL11
- SW51 pad 1: /COL9 -> /COL12
- SW52 pad 1: /COL9 -> /COL13
- SW53 pad 1: /COL9 -> /COL14
- SW54 pad 1: /COL10 -> /COL15
- SW55 pad 1: /COL10 -> /COL16
- SW56 pad 1: /COL10 -> /COL17
- SW57 pad 1: /COL10 -> /COL18
- SW58 pad 1: /COL10 -> /COL19
- SW59 pad 1: /COL10 -> /COL20
- SW6 pad 1: /COL0 -> /COL5
- SW60 pad 1: /COL11 -> /COL0
- SW61 pad 1: /COL11 -> /COL1
- SW62 pad 1: /COL11 -> /COL2
- SW63 pad 1: /COL11 -> /COL3
- SW64 pad 1: /COL11 -> /COL4
- SW65 pad 1: /COL11 -> /COL5
- SW66 pad 1: /COL12 -> /COL6
- SW67 pad 1: /COL12 -> /COL7
- SW68 pad 1: /COL12 -> /COL8
- SW69 pad 1: /COL12 -> /COL9
- SW7 pad 1: /COL1 -> /COL6
- SW70 pad 1: /COL12 -> /COL10
- SW71 pad 1: /COL12 -> /COL11
- SW72 pad 1: /COL13 -> /COL12
- SW73 pad 1: /COL13 -> /COL17
- SW74 pad 1: /COL13 -> /COL18
- SW76 pad 1: /COL14 -> /COL1
- SW77 pad 1: /COL14 -> /COL2
- SW78 pad 1: /COL14 -> /COL3
- SW79 pad 1: /COL14 -> /COL4
- SW8 pad 1: /COL1 -> /COL7
- SW80 pad 1: /COL15 -> /COL5
- SW81 pad 1: /COL15 -> /COL6
- SW82 pad 1: /COL15 -> /COL7
- SW83 pad 1: /COL15 -> /COL8
- SW84 pad 1: /COL15 -> /COL9
- SW85 pad 1: /COL16 -> /COL10
- SW86 pad 1: /COL16 -> /COL11
- SW87 pad 1: /COL16 -> /COL12
- SW88 pad 1: /COL16 -> /COL15
- SW9 pad 1: /COL1 -> /COL8
- SW90 pad 1: /COL17 -> /COL18
- SW91 pad 1: /COL17 -> /COL19
- SW92 pad 1: /COL17 -> /COL20
- SW93 pad 1: /COL17 -> /COL0
- SW94 pad 1: /COL18 -> /COL1
- SW95 pad 1: /COL18 -> /COL2
- SW96 pad 1: /COL18 -> /COL5
- SW97 pad 1: /COL18 -> /COL10
- SW98 pad 1: /COL19 -> /COL11
- SW99 pad 1: /COL19 -> /COL12
- U1 pad 1: unconnected-(U1-3V3-Pad1)_1 -> /unconnected-(U1-3V3-Pad1)_1
- U1 pad 2: unconnected-(U1-3V3-Pad1) -> /unconnected-(U1-3V3-Pad1)_1_1
Routing:
- net (no net): track 0.00 -> 2089.5 mm
- net Net-(U1-GPIO42/MTMS): track 0.00 -> 907.5 mm
- net Net-(U1-GPIO41/MTDI): track 0.00 -> 627.4 mm
- net /COL19: track 0.00 -> 626.6 mm
- net /COL17: track 0.00 -> 617.1 mm
- net /ROW4: track 0.00 -> 584.9 mm
- net /ROW5: track 0.00 -> 583.2 mm
- net Net-(U1-GPIO40/MTDO): track 0.00 -> 569.5 mm
- net /COL20: track 0.00 -> 527.0 mm
- net /ROW3: track 0.00 -> 514.0 mm
- net /ROW2: track 0.00 -> 484.2 mm
- net /COL16: track 0.00 -> 476.3 mm
- net /ROW1: track 0.00 -> 463.0 mm
- net /COL15: track 0.00 -> 438.0 mm
- net GND: track 0.00 -> 437.9 mm
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Other:
- board size 502.4 x 209.1 mm -> 479 x 141.5 mm
