File: Keep-KiCad/keeboard/keeboard.kicad_sch (KiCad schematic)
At the start: 203 parts, among them SW1 SW_Push, SW10 SW_Push, SW100 SW_Push, SW101 RotaryEncoder_Switch, SW11 SW_Push, SW12 SW_Push, SW13 SW_Push, SW14 SW_Push, SW15 SW_Push, SW16 SW_Push, SW17 SW_Push, SW18 SW_Push, SW19 SW_Push, SW2 SW_Push, SW20 SW_Push, SW21 SW_Push, SW22 SW_Push, SW23 SW_Push, SW24 SW_Push, SW25 SW_Push, SW26 SW_Push, SW27 SW_Push, SW28 SW_Push, SW29 SW_Push, SW3 SW_Push, SW30 SW_Push, SW31 SW_Push, SW32 SW_Push, SW33 SW_Push, SW34 SW_Push, SW35 SW_Push, SW36 SW_Push, SW37 SW_Push, SW38 SW_Push, SW39 SW_Push, SW4 SW_Push, SW40 SW_Push, SW41 SW_Push, SW42 SW_Push, SW43 SW_Push, SW44 SW_Push, SW45 SW_Push, SW46 SW_Push, SW47 SW_Push, SW48 SW_Push, SW49 SW_Push, SW5 SW_Push, SW50 SW_Push, SW51 SW_Push, SW52 SW_Push, SW53 SW_Push, SW54 SW_Push, SW55 SW_Push, SW56 SW_Push, SW57 SW_Push, SW58 SW_Push, SW59 SW_Push, SW6 SW_Push, SW60 SW_Push, SW61 SW_Push, SW62 SW_Push, SW63 SW_Push, SW64 SW_Push, SW65 SW_Push, SW66 SW_Push, SW67 SW_Push, SW68 SW_Push, SW69 SW_Push, SW7 SW_Push, SW70 SW_Push, SW71 SW_Push, SW72 SW_Push, SW73 SW_Push, SW74 SW_Push, SW75 SW_Push, SW76 SW_Push, SW77 SW_Push, SW78 SW_Push, SW79 SW_Push, SW8 SW_Push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

Commit message: updating pcb stuff
Parts:
- removed A1: RaspberryPi_Pico, Module:RaspberryPi_Pico_Common_Unspecified, symbol MCU_Module:RaspberryPi_Pico
- removed D5, D6, D69, D70, D74: 1N4148, Diode_THT:D_DO-35_SOD27_P7.62mm_Horizontal, symbol Diode:1N4148
- removed SW101: RotaryEncoder_Switch, symbol Device:RotaryEncoder_Switch
- removed SW5, SW6, SW69, SW70, SW74: SW_Push, symbol Switch:SW_Push
- added D101, D102, D103, D104, D75, D78, D79, D80, D81: 1N4148, Diode_THT:D_DO-35_SOD27_P7.62mm_Horizontal, symbol Diode:1N4148
- added S2, S3, S4: MX_stab, PCM_marbastlib-mx:STAB_MX_2u, symbol PCM_marbastlib-mx:MX_stab
- added S5: MX_stab, PCM_marbastlib-mx:STAB_MX_2.25u, symbol PCM_marbastlib-mx:MX_stab
- added S6: MX_stab, PCM_marbastlib-mx:STAB_MX_2.75u, symbol PCM_marbastlib-mx:MX_stab
- added S7: MX_stab, PCM_marbastlib-mx:STAB_MX_6.25u, symbol PCM_marbastlib-mx:MX_stab
- added SW1: RotaryEncoder_Switch, Rotary_Encoder:RotaryEncoder_Alps_EC11E-Switch_Vertical_H20mm, symbol Device:RotaryEncoder_Switch
- added SW101, SW102, SW103, SW104, SW105, SW78, SW80, SW81: SW_Push, PCM_marbastlib-mx:SW_MX_HS_CPG151101S11_1u, symbol Switch:SW_Push
- added SW79: SW_Push, PCM_marbastlib-mx:SW_MX_HS_CPG151101S11_1.25u, symbol Switch:SW_Push
- added U1: ESP32-S3-DevKitC, PCM_Espressif:ESP32-S3-DevKitC, symbol PCM_Espressif:ESP32-S3-DevKitC
- S1: footprint PCM_marbastlib-mx:STAB_MX_P_6.25u -> PCM_marbastlib-mx:STAB_MX_2u
- SW10, SW100, SW7, SW76, SW77, SW8, SW82, SW83, SW85, SW86, SW87, SW89, SW9, SW90, SW91, SW92, SW94, SW95, SW96, SW97, SW98, SW99: footprint (none) -> PCM_marbastlib-mx:SW_MX_HS_CPG151101S11_1u
- SW11: renamed from SW72; footprint (none) -> PCM_marbastlib-mx:SW_MX_HS_CPG151101S11_1.25u
- SW12: renamed from SW11; footprint (none) -> PCM_marbastlib-mx:SW_MX_HS_CPG151101S11_1u
- SW13: renamed from SW12; footprint (none) -> PCM_marbastlib-mx:SW_MX_HS_CPG151101S11_1u
- SW14: renamed from SW13; footprint (none) -> PCM_marbastlib-mx:SW_MX_HS_CPG151101S11_1u
- SW15: renamed from SW14; footprint (none) -> PCM_marbastlib-mx:SW_MX_HS_CPG151101S11_1u
- SW16: renamed from SW15; footprint (none) -> PCM_marbastlib-mx:SW_MX_HS_CPG151101S11_1u
- SW17: renamed from SW73; footprint (none) -> PCM_marbastlib-mx:SW_MX_HS_CPG151101S11_1.25u
- SW18: renamed from SW16; footprint (none) -> PCM_marbastlib-mx:SW_MX_HS_CPG151101S11_1u
- SW19: renamed from SW17; footprint (none) -> PCM_marbastlib-mx:SW_MX_HS_CPG151101S11_1u
- SW2: renamed from SW1; footprint (none) -> PCM_marbastlib-mx:SW_MX_HS_CPG151101S11_1u
- SW20: renamed from SW18; footprint (none) -> PCM_marbastlib-mx:SW_MX_HS_CPG151101S11_1u
- SW21: renamed from SW19; footprint (none) -> PCM_marbastlib-mx:SW_MX_HS_CPG151101S11_1u
- SW22: renamed from SW20; footprint (none) -> PCM_marbastlib-mx:SW_MX_HS_CPG151101S11_1u
- SW23: renamed from SW21; footprint (none) -> PCM_marbastlib-mx:SW_MX_HS_CPG151101S11_1u
- SW24: renamed from SW22; footprint (none) -> PCM_marbastlib-mx:SW_MX_HS_CPG151101S11_1u
- SW25: renamed from SW23; footprint (none) -> PCM_marbastlib-mx:SW_MX_HS_CPG151101S11_1u
- SW26: renamed from SW24; footprint (none) -> PCM_marbastlib-mx:SW_MX_HS_CPG151101S11_1u
- SW27: renamed from SW25; footprint (none) -> PCM_marbastlib-mx:SW_MX_HS_CPG151101S11_1u
- SW28: renamed from SW26; footprint (none) -> PCM_marbastlib-mx:SW_MX_HS_CPG151101S11_1u
- SW29: renamed from SW27; footprint (none) -> PCM_marbastlib-mx:SW_MX_HS_CPG151101S11_1u
- SW3: renamed from SW2; footprint (none) -> PCM_marbastlib-mx:SW_MX_HS_CPG151101S11_1.5u
- SW30: renamed from SW28; footprint (none) -> PCM_marbastlib-mx:SW_MX_HS_CPG151101S11_1u
- SW31: renamed from SW29; footprint (none) -> PCM_marbastlib-mx:SW_MX_HS_CPG151101S11_1u
- SW32: renamed from SW30; footprint (none) -> PCM_marbastlib-mx:SW_MX_HS_CPG151101S11_1u
- SW33: renamed from SW75; footprint (none) -> PCM_marbastlib-mx:SW_MX_HS_CPG151101S11_1u
- SW34: renamed from SW31; footprint (none) -> PCM_marbastlib-mx:SW_MX_HS_CPG151101S11_1u
- SW35: renamed from SW32; footprint (none) -> PCM_marbastlib-mx:SW_MX_HS_CPG151101S11_1u
- SW36: renamed from SW33; footprint (none) -> PCM_marbastlib-mx:SW_MX_HS_CPG151101S11_1u
- SW37: renamed from SW34; footprint (none) -> PCM_marbastlib-mx:SW_MX_HS_CPG151101S11_1u
- SW38: renamed from SW35; footprint (none) -> PCM_marbastlib-mx:SW_MX_HS_CPG151101S11_1u
- SW39: renamed from SW36; footprint (none) -> PCM_marbastlib-mx:SW_MX_HS_CPG151101S11_1u
- SW4: renamed from SW3; footprint (none) -> PCM_marbastlib-mx:SW_MX_HS_CPG151101S11_1.75u
- SW40: renamed from SW37; footprint (none) -> PCM_marbastlib-mx:SW_MX_HS_CPG151101S11_1u
- SW41: renamed from SW38; footprint (none) -> PCM_marbastlib-mx:SW_MX_HS_CPG151101S11_1u
- SW42: renamed from SW39; footprint (none) -> PCM_marbastlib-mx:SW_MX_HS_CPG151101S11_1u
- SW43: renamed from SW40; footprint (none) -> PCM_marbastlib-mx:SW_MX_HS_CPG151101S11_1u
- SW44: renamed from SW41; footprint (none) -> PCM_marbastlib-mx:SW_MX_HS_CPG151101S11_1u
- SW45: renamed from SW42; footprint (none) -> PCM_marbastlib-mx:SW_MX_HS_CPG151101S11_1u
- SW46: renamed from SW43; footprint (none) -> PCM_marbastlib-mx:SW_MX_HS_CPG151101S11_1u
- SW47: renamed from SW44; footprint (none) -> PCM_marbastlib-mx:SW_MX_HS_CPG151101S11_1u
- SW48: renamed from SW45; footprint (none) -> PCM_marbastlib-mx:SW_MX_HS_CPG151101S11_1u
- SW49: renamed from SW46; footprint (none) -> PCM_marbastlib-mx:SW_MX_HS_CPG151101S11_1u
- SW5: renamed from SW4; footprint (none) -> PCM_marbastlib-mx:SW_MX_HS_CPG151101S11_1u
- SW50: renamed from SW47; footprint (none) -> PCM_marbastlib-mx:SW_MX_HS_CPG151101S11_1u
- SW51: renamed from SW48; footprint (none) -> PCM_marbastlib-mx:SW_MX_HS_CPG151101S11_1u
- SW52: renamed from SW49; footprint (none) -> PCM_marbastlib-mx:SW_MX_HS_CPG151101S11_1u
- SW53: renamed from SW50; footprint (none) -> PCM_marbastlib-mx:SW_MX_HS_CPG151101S11_1u
- SW54: renamed from SW51; footprint (none) -> PCM_marbastlib-mx:SW_MX_HS_CPG151101S11_1u
- SW55: renamed from SW52; footprint (none) -> PCM_marbastlib-mx:SW_MX_HS_CPG151101S11_1u
- SW56: renamed from SW53; footprint (none) -> PCM_marbastlib-mx:SW_MX_HS_CPG151101S11_1u
- SW57: renamed from SW54; footprint (none) -> PCM_marbastlib-mx:SW_MX_HS_CPG151101S11_1u
- SW58: renamed from SW55; footprint (none) -> PCM_marbastlib-mx:SW_MX_HS_CPG151101S11_1u
- SW59: renamed from SW78; footprint (none) -> PCM_marbastlib-mx:SW_MX_HS_CPG151101S11_1u
- SW6: renamed from SW71; footprint (none) -> PCM_marbastlib-mx:SW_MX_HS_CPG151101S11_1.25u
- SW60: renamed from SW56; footprint (none) -> PCM_marbastlib-mx:SW_MX_HS_CPG151101S11_1u
- SW61: renamed from SW57; footprint (none) -> PCM_marbastlib-mx:SW_MX_HS_CPG151101S11_1u
- SW62: renamed from SW58; footprint (none) -> PCM_marbastlib-mx:SW_MX_HS_CPG151101S11_1u
- SW63: renamed from SW59; footprint (none) -> PCM_marbastlib-mx:SW_MX_HS_CPG151101S11_1u
- SW64: renamed from SW60; footprint (none) -> PCM_marbastlib-mx:SW_MX_HS_CPG151101S11_1u
- SW65: renamed from SW79; footprint (none) -> PCM_marbastlib-mx:SW_MX_HS_CPG151101S11_1u
- SW66: renamed from SW61; footprint (none) -> PCM_marbastlib-mx:SW_MX_HS_CPG151101S11_1u
- SW67: renamed from SW62; footprint (none) -> PCM_marbastlib-mx:SW_MX_HS_CPG151101S11_1u
- SW68: renamed from SW63; footprint (none) -> PCM_marbastlib-mx:SW_MX_HS_CPG151101S11_1u
- SW69: renamed from SW64; footprint (none) -> PCM_marbastlib-mx:SW_MX_HS_CPG151101S11_1u
- SW70: renamed from SW65; footprint (none) -> PCM_marbastlib-mx:SW_MX_HS_CPG151101S11_1u
- SW71: renamed from SW80; footprint (none) -> PCM_marbastlib-mx:SW_MX_HS_CPG151101S11_1u
- SW72: renamed from SW66; footprint (none) -> PCM_marbastlib-mx:SW_MX_HS_CPG151101S11_1.5u
- SW73: renamed from SW67; footprint (none) -> PCM_marbastlib-mx:SW_MX_HS_CPG151101S11_1u
- SW74: renamed from SW68; footprint (none) -> PCM_marbastlib-mx:SW_MX_HS_CPG151101S11_1u
- SW75: renamed from SW81; footprint (none) -> PCM_marbastlib-mx:SW_MX_HS_CPG151101S11_1u
- SW84, SW88, SW93: footprint (none) -> PCM_marbastlib-mx:SW_MX_HS_CPG151101S11_1.25u
- renumbered D72 to D10, D73 to D16, D16 to D17, D17 to D18, D18 to D19, D19 to D20, D20 to D21, D21 to D22, D22 to D23, D23 to D24, D24 to D25, D25 to D26, D26 to D27, D27 to D28, D28 to D29, D29 to D30, D30 to D31, D75 to D32, D31 to D33, D32 to D34, D33 to D35, D34 to D36, D35 to D37, D36 to D38, D37 to D39, D38 to D40, D39 to D41, D40 to D42, D41 to D43, D42 to D44, D43 to D45, D44 to D46, D45 to D47, D46 to D48, D47 to D49, D71 to D5, D48 to D50, D49 to D51, D50 to D52, D51 to D53, D52 to D54, D53 to D55, D54 to D56, D55 to D57, D78 to D58, D56 to D59, D7 to D6, D57 to D60, D58 to D61, D59 to D62, D60 to D63, D79 to D64, D61 to D65, D62 to D66, D63 to D67, D64 to D68, D65 to D69, D8 to D7, D80 to D70, D66 to D71, D67 to D72, D68 to D73, D81 to D74, D9 to D8, D10 to D9
Connections:
- net ROW2: now reaches D61.1 (K)
- net ROW2: now also D13.1 (K), D19.1 (K), D24.1 (K), D29.1 (K), D3.1 (K), D35.1 (K), D40.1 (K), D45.1 (K), D50.1 (K), D55.1 (K), D67.1 (K), D7.1 (K), D73.1 (K), D77.1 (K), D86.1 (K), D89.1 (K), D94.1 (K), D98.1 (K), D103.1 (K), D81.1 (K)
- net ROW1: now reaches D34.1 (K)
- net ROW1: now also D12.1 (K), D18.1 (K), D2.1 (K), D23.1 (K), D28.1 (K), D39.1 (K), D44.1 (K), D49.1 (K), D54.1 (K), D6.1 (K), D60.1 (K), D66.1 (K), D72.1 (K), D76.1 (K), D85.1 (K), D88.1 (K), D93.1 (K), D97.1 (K), D102.1 (K), D80.1 (K)
- net ROW3: now reaches D30.1 (K)
- net ROW3: now also D14.1 (K), D20.1 (K), D25.1 (K), D36.1 (K), D4.1 (K), D41.1 (K), D46.1 (K), D51.1 (K), D56.1 (K), D62.1 (K), D68.1 (K), D8.1 (K), D90.1 (K), D95.1 (K), D99.1 (K)
- net ROW0: now reaches D17.1 (K)
- net ROW0: now also D1.1 (K), D11.1 (K), D22.1 (K), D27.1 (K), D33.1 (K), D38.1 (K), D43.1 (K), D48.1 (K), D53.1 (K), D59.1 (K), D65.1 (K), D71.1 (K), D84.1 (K), D75.1 (K), D79.1 (K)
- net at SW99.2: now also D98.2 (A); no longer D99.2 (A)
- net at D97.2 (A): now also SW98.2; no longer SW97.2
- net ROW5: now reaches D64.1 (K)
- net ROW5: now also D10.1 (K), D16.1 (K), D32.1 (K), D5.1 (K), D58.1 (K), D70.1 (K), D74.1 (K), D83.1 (K), D87.1 (K), D92.1 (K), D101.1 (K), D78.1 (K)
- net at D96.2 (A): now also SW97.2; no longer SW96.2
- net at D93.2 (A): now also SW94.2; no longer SW93.2
- net at D76.2 (A): now also SW77.2; no longer SW76.2
- net at D77.2 (A): now also SW78.2; no longer SW77.2
- net ROW4: now reaches D42.1 (K)
- net ROW4: now also D100.1 (K), D15.1 (K), D21.1 (K), D26.1 (K), D31.1 (K), D37.1 (K), D47.1 (K), D52.1 (K), D57.1 (K), D63.1 (K), D69.1 (K), D82.1 (K), D9.1 (K), D91.1 (K), D96.1 (K), D104.1 (K)
- net at SW100.2: now also D99.2 (A); no longer D100.2 (A)
- net at SW82.2: now also D81.2 (A)
- net at SW92.2: now also D91.2 (A); no longer D92.2 (A)
- net at SW87.2: now also D86.2 (A)
- net at SW84.2: now also D83.2 (A)
- net at D94.2 (A): now also SW95.2; no longer SW94.2
- net at SW91.2: now also D90.2 (A); no longer D91.2 (A)
- net at SW85.2: now also D84.2 (A)
- net at SW89.2: now also D88.2 (A)
- net at SW86.2: now also D85.2 (A)
- net at D87.2 (A): now also SW88.2
- net at SW90.2: now also D89.2 (A)
- net at D95.2 (A): now also SW96.2; no longer SW95.2
- net at D82.2 (A): now also SW83.2
- net COL 0 renamed COL0
- net COL 07 renamed COL7
- net COL7: no longer SW76.1
- net COL 1 renamed COL1
- net COL 10 renamed COL10
- net COL 11 renamed COL11
- net COL 12 renamed COL12
- net COL 13 renamed COL13
- net COL 14 renamed COL16
- net COL16: now also SW86.1, SW87.1, U1.30 (GPIO45); no longer SW82.1, SW91.1
- removed net COL 15: SW83.1, SW86.1, SW89.1, SW92.1, SW94.1
- net COL 16 renamed COL17
- net COL17: now also SW89.1, SW91.1, SW92.1, U1.14 (GPIO46); no longer SW84.1, SW87.1
- net COL 17 renamed COL18
- net COL18: now also SW94.1, U1.28 (GPIO47); no longer SW100.1, SW98.1, SW99.1
- net COL 2 renamed COL2
- net COL 3 renamed COL3
- net COL 4 renamed COL4
- net COL 5 renamed COL5
- net COL 6 renamed COL6
- net COL 8 renamed COL8
- net COL 9 renamed COL9
- net COL9: no longer SW77.1
- new net: D102.2 (A), SW103.2
- new net: D104.2 (A), SW105.2
- new net: D101.2 (A), SW102.2
- new net: SW1.A, U1.37 (GPIO40/MTDO)
- new net: SW1.B, U1.38 (GPIO41/MTDI)
- new net: SW1.S1, U1.39 (GPIO42/MTMS)
- new net: D79.2 (A), SW80.2
- new net: D92.2 (A), SW93.2
- new net: D103.2 (A), SW104.2
- new net: D78.2 (A), SW79.2
- new net: D100.2 (A), SW101.2
- new net: D75.2 (A), SW76.2
- new net: D80.2 (A), SW81.2
- new net: U1.1 (3V3), U1.2 (3V3)
- new net COL14: SW76.1, SW77.1, SW78.1, SW79.1, U1.34 (GPIO37)
- new net COL15: SW80.1, SW81.1, SW82.1, SW83.1, SW84.1, U1.35 (GPIO38)
- new net COL19: SW100.1, SW101.1, SW102.1, SW98.1, SW99.1, U1.29 (GPIO48)
- new net COL20: SW103.1, SW104.1, SW105.1, U1.36 (GPIO39/MTCK)
- new net GND: SW1.C, SW1.S2, U1.22 (GND), U1.23 (GND), U1.24 (GND), U1.44 (GND)
Other:
- moved on the sheet: S1

Commit message: pcb edit & schematic
Parts:
- added S8: MX_stab, PCM_marbastlib-mx:STAB_MX_2u, symbol PCM_marbastlib-mx:MX_stab
- D1, D10, D100, D101, D102, D103, D104, D11, D12, D13, D14, D15, D16, D17, D18, D19, D2, D20, D21, D22, D23, D24, D25, D26, D27, D28, D29, D3, D30, D31, D32, D33, D34, D35, D36, D37, D38, D39, D4, D40, D41, D42, D43, D44, D45, D46, D47, D48, D49, D5, D50, D51, D52, D53, D54, D55, D56, D57, D58, D59, D6, D60, D61, D62, D63, D64, D65, D66, D67, D68, D69, D7, D70, D71, D72, D73, D75, D76, D77, D78, D79, D8, D80, D81, D82, D83, D84, D85, D86, D87, D88, D89, D9, D90, D91, D92, D93, D94, D95, D96, D97, D98, D99: KiLib_Generator (none) -> diode/THT
- S1, S2, S3, S4, S5, S6, S7: now left out of the parts list
- SW17, SW79, SW84: footprint PCM_marbastlib-mx:SW_MX_HS_CPG151101S11_1.25u -> PCM_marbastlib-mx:SW_MX_HS_CPG151101S11_1u
- SW72: footprint PCM_marbastlib-mx:SW_MX_HS_CPG151101S11_1.5u -> PCM_marbastlib-mx:SW_MX_HS_CPG151101S11_1u
Connections:
- net COL0: now also U1.6 (GPIO6/ADC1_CH5)
- net COL1: now also U1.7 (GPIO7/ADC1_CH6)
- net COL10: now also U1.11 (GPIO18/ADC2_CH7)
- net COL11: now also U1.27 (GPIO21)
- net COL12: now also U1.32 (GPIO35)
- net COL13: now also U1.33 (GPIO36)
- net COL2: now also U1.12 (GPIO8/ADC1_CH7)
- net COL3: now also U1.15 (GPIO9/ADC1_CH8)
- net COL4: now also U1.16 (GPIO10/ADC1_CH9)
- net COL5: now also U1.17 (GPIO11/ADC2_CH0)
- net COL6: now also U1.18 (GPIO12/ADC2_CH1)
- net COL7: now also U1.19 (GPIO13/ADC2_CH2)
- net COL8: now also U1.20 (GPIO14/ADC2_CH3)
- net COL9: now also U1.10 (GPIO17/ADC2_CH6)
- net ROW0: now also U1.31 (GPIO0)
- net ROW1: now also U1.41 (GPIO1/ADC1_CH0)
- net ROW2: now also U1.40 (GPIO2/ADC1_CH1)
- net ROW3: now also U1.13 (GPIO3/ADC1_CH2)
- net ROW4: now also U1.4 (GPIO4/ADC1_CH3)
- net ROW5: now also U1.5 (GPIO5/ADC1_CH4)
- net unconnected-(U1-3V3-Pad1)_1: now reaches U1.1 (3V3), U1.2 (3V3)
- no-connect marks 0 -> 9

Commit message: Finishing up the pcb
did all routing, wiring, etc...
Parts:
- renumbered D53 to D10, D78 to D100, D83 to D101, D87 to D102, D92 to D103, D101 to D104, D59 to D11, D65 to D12, D71 to D13, D75 to D14, D79 to D15, D84 to D16, D2 to D17, D6 to D18, D12 to D19, D11 to D2, D18 to D20, D23 to D21, D28 to D22, D34 to D23, D39 to D24, D44 to D25, D49 to D26, D54 to D27, D60 to D28, D66 to D29, D17 to D3, D72 to D30, D76 to D31, D80 to D32, D85 to D33, D88 to D34, D93 to D35, D97 to D36, D102 to D37, D3 to D38, D7 to D39, D22 to D4, D13 to D40, D19 to D41, D24 to D42, D29 to D43, D35 to D44, D40 to D45, D45 to D46, D50 to D47, D55 to D48, D61 to D49, D27 to D5, D67 to D50, D73 to D51, D77 to D52, D81 to D53, D86 to D54, D89 to D55, D94 to D56, D98 to D57, D103 to D58, D4 to D59, D33 to D6, D8 to D60, D14 to D61, D20 to D62, D25 to D63, D30 to D64, D36 to D65, D41 to D66, D46 to D67, D51 to D68, D56 to D69, D38 to D7, D62 to D70, D68 to D71, D90 to D72, D95 to D73, D99 to D74, D9 to D75, D15 to D76, D21 to D77, D26 to D78, D31 to D79, D43 to D8, D37 to D80, D42 to D81, D47 to D82, D52 to D83, D57 to D84, D63 to D85, D69 to D86, D82 to D87, D91 to D88, D96 to D89, D48 to D9, D100 to D90, D104 to D91, D5 to D92, D10 to D93, D16 to D94, D32 to D95, D58 to D96, D64 to D97, D70 to D98, D74 to D99, SW49 to SW10, SW75 to SW100, SW79 to SW101, SW84 to SW102, SW88 to SW103, SW93 to SW104, SW102 to SW105, SW54 to SW11, SW60 to SW12, SW66 to SW13, SW72 to SW14, SW76 to SW15, SW80 to SW16, SW85 to SW17, SW3 to SW18, SW7 to SW19, SW13 to SW20, SW19 to SW21, SW24 to SW22, SW29 to SW23, SW35 to SW24, SW40 to SW25, SW45 to SW26, SW50 to SW27, SW55 to SW28, SW61 to SW29, SW12 to SW3, SW67 to SW30, SW73 to SW31, SW77 to SW32, SW81 to SW33, SW86 to SW34, SW89 to SW35, SW94 to SW36, SW98 to SW37, SW103 to SW38, SW4 to SW39, SW18 to SW4, SW8 to SW40, SW14 to SW41, SW20 to SW42, SW25 to SW43, SW30 to SW44, SW36 to SW45, SW41 to SW46, SW46 to SW47, SW51 to SW48, SW56 to SW49, SW23 to SW5, SW62 to SW50, SW68 to SW51, SW74 to SW52, SW78 to SW53, SW82 to SW54, SW87 to SW55, SW90 to SW56, SW95 to SW57, SW99 to SW58, SW104 to SW59, SW28 to SW6, SW5 to SW60, SW9 to SW61, SW15 to SW62, SW21 to SW63, SW26 to SW64, SW31 to SW65, SW37 to SW66, SW42 to SW67, SW47 to SW68, SW52 to SW69, SW34 to SW7, SW57 to SW70, SW63 to SW71, SW69 to SW72, SW91 to SW73, SW96 to SW74, SW100 to SW75, SW10 to SW76, SW16 to SW77, SW22 to SW78, SW27 to SW79, SW39 to SW8, SW32 to SW80, SW38 to SW81, SW43 to SW82, SW48 to SW83, SW53 to SW84, SW58 to SW85, SW64 to SW86, SW70 to SW87, SW83 to SW88, SW92 to SW89, SW44 to SW9, SW97 to SW90, SW101 to SW91, SW105 to SW92, SW6 to SW93, SW11 to SW94, SW17 to SW95, SW33 to SW96, SW59 to SW97, SW65 to SW98, SW71 to SW99
